File: ErgoBoard.kicad_pcb (KiCad board)
At the start: 2 copper layers, 157 x 119 mm, 69 parts, among them SW1 SW_Push, SW10 SW_Push, SW11 SW_Push, SW12 SW_Push, SW13 SW_Push, SW14 SW_Push, SW15 SW_Push, SW16 SW_Push, SW17 SW_Push, SW18 SW_Push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

Commit message: Add UART debug test points
Parts:
- added J1: Conn_01x03_Pin, Connector_PinHeader_2.54mm:PinHeader_1x03_P2.54mm_Vertical, F.Cu at (254.6, 43.8)
- renumbered JackL1 to Link, JackR1 to Zelda
Routing:
- net UART_TX: track 105.4 -> 135.3 mm
- net UART_RX: track 105.2 -> 135.1 mm
- net GND: track 135.5 -> 142.9 mm
